Commit message: Update urdf

File: src/diego_nav/description/diego1.urdf (robot description, URDF)
Before this commit: robot diego1, 83 links, 82 joints
Links:
- removed link body
- removed link left_arm_stevo
- removed link left_arm_stevo_axis
- removed link left_big_arm_down
- removed link left_big_arm_up
- removed link left_finger
- removed link left_hand_run_stevo
- removed link left_hand_run_stevo_axis
- removed link left_shoulder_stevo
- removed link left_shoulder_stevo_axis
- removed link left_shoulder_stevo_lift
- removed link left_shoulder_stevo_lift_axis
- removed link left_small_arm_down
- removed link left_small_arm_middle
- removed link left_small_arm_up
- removed link left_wrist_run_stevo
- removed link left_wrist_run_stevo_axis
- removed link left_wrist_stevo
- removed link left_wrist_stevo_axis
- removed link right_arm_stevo
- removed link right_arm_stevo_axis
- removed link right_big_arm_down
- removed link right_big_arm_up
- removed link right_finger
- removed link right_hand_run_stevo
- removed link right_hand_run_stevo_axis
- removed link right_shoulder_stevo
- removed link right_shoulder_stevo_axis
- removed link right_shoulder_stevo_lift
- removed link right_shoulder_stevo_lift_axis
- removed link right_small_arm_down
- removed link right_small_arm_middle
- removed link right_small_arm_up
- removed link right_wrist_run_stevo
- removed link right_wrist_run_stevo_axis
- removed link right_wrist_stevo
- removed link right_wrist_stevo_axis
- added link arm_base; visual box size=0.11 .11 .013
- added link arm_joint_stevo1; visual cylinder length=.09 radius=0.025
- added link arm_joint_stevo2; visual cylinder length=.06 radius=0.025
- added link arm_joint_stevo3; visual cylinder length=.12 radius=0.012
- added link arm_joint_stevo4; visual cylinder length=.05 radius=0.02
- added link arm_joint_stevo5; visual cylinder length=.04 radius=0.02
- added link arm_round_joint_stevo0; visual cylinder length=.013 radius=0.05
- added link big_arm; visual box size=0.05 .05 .13
- added link camera_holder; visual box size=0.043 .03 .59
- added link control_box; visual box size=0.16 .128 .14
- added link finger_left_big; visual box size=0.04 .009 .045
- added link finger_left_small; visual box size=0.04 .009 .045
- added link finger_right_big; visual box size=0.04 .009 .045
- added link finger_right_small; visual box size=0.04 .009 .045
- added link grip_joint_stevo6; visual cylinder length=.05 radius=0.005
- added link grip_joint_stevo7; visual cylinder length=.05 radius=0.005
- added link hand; visual box size=0.04 .06 .02
- added link shoulder_1; visual box size=0.065 .065 .037
- added link shoulder_2; visual box size=0.05 .065 .105
- added link wrist; visual box size=0.045 .04 .06
Joints:
- removed joint base_to_body
- removed joint body_to_left_shoulder_stevo
- removed joint body_to_right_shoulder_stevo
- removed joint body_to_xtion_camera_base
- removed joint left_arm_stevo_to_left_small_arm_up
- removed joint left_big_arm_up_to_axis
- removed joint left_big_arm_up_to_axis_to_left_arm_stevo
- removed joint left_big_arm_up_to_left_big_arm_down
- removed joint left_hand_run_stevo_axis_to_left_finger
- removed joint left_hand_run_stevo_to_left_hand_run_stevo_axis
- removed joint left_shoulder_stevo_axis_to_lift_stevo
- removed joint left_shoulder_stevo_lift_axis_to_left_big_arm
- removed joint left_shoulder_stevo_lift_to_axis
- removed joint left_shoulder_stevo_to_axis
- removed joint left_small_arm_up_to_axis
- removed joint left_small_arm_up_to_axis_to_left_axis_stevo
- removed joint left_small_arm_up_to_left_small_arm_down
- removed joint left_small_arm_up_to_left_small_arm_middle
- removed joint left_wrist_run_stevo_axis_to_left_hand_run_stevo
- removed joint left_wrist_run_stevo_to_axis
- removed joint right_arm_stevo_to_right_small_arm_up
- removed joint right_big_arm_up_to_axis
- removed joint right_big_arm_up_to_axis_to_right_arm_stevo
- removed joint right_big_arm_up_to_right_big_arm_down
- removed joint right_hand_run_stevo_axis_to_right_finger
- removed joint right_hand_run_stevo_to_right_hand_run_stevo_axis
- removed joint right_shoulder_stevo_axis_to_lift_stevo
- removed joint right_shoulder_stevo_lift_axis_to_right_big_arm
- removed joint right_shoulder_stevo_lift_to_axis
- removed joint right_shoulder_stevo_to_axis
- removed joint right_small_arm_up_to_axis
- removed joint right_small_arm_up_to_axis_to_right_axis_stevo
- removed joint right_small_arm_up_to_right_small_arm_down
- removed joint right_small_arm_up_to_right_small_arm_middle
- removed joint right_wrist_run_stevo_axis_to_right_hand_run_stevo
- removed joint right_wrist_run_stevo_to_axis
- removed joint right_wrist_stevo_to_left_wrist_run_stevo
- removed joint right_wrist_stevo_to_right_wrist_run_stevo
- added joint arm_base_to_arm_round_joint_stevo0: type revolute, parent arm_base, child arm_round_joint_stevo0, origin xyz=0.00 0.00 0.013 rpy=0 0 0, axis 0 0 1, limit lower=-1.5707963 upper=1.5707963 effort=100 velocity=100
- added joint arm_joint_stevo1_to_big_arm: type fixed, parent arm_joint_stevo1, child big_arm, origin xyz=0.0 0.065 0.0 rpy=1.5707963 0 0
- added joint arm_joint_stevo2_to_arm_joint_stevo3: type revolute, parent arm_joint_stevo2, child arm_joint_stevo3, origin xyz=0.00 -0.06 0.00 rpy=1.5707963 -0.52359877 0, axis 0 0 1, limit lower=-1.5707963 upper=1.5707963 effort=100 velocity=100
- added joint arm_joint_stevo3_to_wrist: type fixed, parent arm_joint_stevo3, child wrist, origin xyz=0.0 0.0 0.09 rpy=0 0 0
- added joint arm_joint_stevo4_to_arm_joint_stevo5: type revolute, parent arm_joint_stevo4, child arm_joint_stevo5, origin xyz=-0.02 0.00 0.00 rpy=0 1.5707963 0, axis 0 0 1, limit lower=-1.5707963 upper=1.5707963 effort=100 velocity=100
- added joint arm_joint_stevo5_to_hand: type fixed, parent arm_joint_stevo5, child hand, origin xyz=0.0 0.0 -0.03 rpy=0 0 0
- added joint arm_round_joint_stevo0_to_shoulder_1: type fixed, parent arm_round_joint_stevo0, child shoulder_1, origin xyz=0.0 0.0 0.025
- added joint base_to_arm_base: type fixed, parent base_link, child arm_base, origin xyz=0.085 0.0 0.008
- added joint base_to_control_box: type fixed, parent base_link, child control_box, origin xyz=-0.07 0.0 0.0715
- added joint big_arm_round_to_joint_stevo2: type revolute, parent big_arm, child arm_joint_stevo2, origin xyz=0.00 0.00 -0.065 rpy=1.5707963 0 0, axis 0 0 1, limit lower=1.0 upper=2.5891 effort=100 velocity=100
- added joint camera_holder_to_xtion_camera_base: type fixed, parent camera_holder, child xtion_camera_base, origin xyz=0.0 0.0 0.3075
- added joint control_box_to_camera_holder: type fixed, parent control_box, child camera_holder, origin xyz=-0.0215 0.0 0.365
- added joint finger_left_big_to_finger_left_small: type fixed, parent finger_left_big, child finger_left_small, origin xyz=0.04 -0.008 0.0 rpy=0 0 -0.34906585
- added joint finger_right_big_to_finger_right_small: type fixed, parent finger_right_big, child finger_right_small, origin xyz=0.04 0.008 0.0 rpy=0 0 0.34906585
- added joint grip_joint_stevo6_to_finger_left_big: type fixed, parent grip_joint_stevo6, child finger_left_big, origin xyz=0.03 0.0 0.0 rpy=0 0 0.34906585
- added joint grip_joint_stevo7_to_finger_right_big: type fixed, parent grip_joint_stevo7, child finger_right_big, origin xyz=0.03 0.0 0.0 rpy=0 0 -0.34906585
- added joint hand_to_grip_joint_stevo6: type revolute, parent hand, child grip_joint_stevo6, origin xyz=0.00 0.015 0.00 rpy=0 1.5707963 0, axis 0 0 1, limit lower=-0.1762 upper=0.8285 effort=100 velocity=100
- added joint hand_to_grip_joint_stevo7: type revolute, parent hand, child grip_joint_stevo7, origin xyz=0.00 -0.015 0.00 rpy=0 1.5707963 0, axis 0 0 1, limit lower=-0.8285 upper=0.1584 effort=100 velocity=100
- added joint shoulder_1_to_shoulder_1: type fixed, parent shoulder_1, child shoulder_2, origin xyz=0.022 0.0 0.03915 rpy=0 0.785398 0
- added joint shoulder_2_to_arm_joint_stevo1: type revolute, parent shoulder_2, child arm_joint_stevo1, origin xyz=0.00 0.00 0.025 rpy=1.5707963 0 0, axis 0 0 1, limit lower=-0.1899 upper=1.5707963 effort=100 velocity=100
- added joint wrist_to_arm_joint_stevo4: type revolute, parent wrist, child arm_joint_stevo4, origin xyz=0.00 0.00 0.03 rpy=0 1.5707963 0, axis 0 0 1, limit lower=-1.5707963 upper=1.5707963 effort=100 velocity=100

Commit message: fix bug

File: src/diego_nav/description/diego1.urdf (robot description, URDF)
Before this commit: robot diego1, 66 links, 65 joints
Joints:
- joint left_leg_to_master_left_axis: type fixed -> continuous
- joint right_leg_to_master_right_axix: type fixed -> continuous
- joint right_leg_to_slave_left_axix1: type fixed -> continuous
- joint right_leg_to_slave_left_axix2: type fixed -> continuous
- joint right_leg_to_slave_left_axix3: type fixed -> continuous
- joint right_leg_to_slave_left_axix4: type fixed -> continuous
- joint right_leg_to_slave_left_axix5: type fixed -> continuous
- joint right_leg_to_slave_right_axix1: type fixed -> continuous
- joint right_leg_to_slave_right_axix2: type fixed -> continuous
- joint right_leg_to_slave_right_axix3: type fixed -> continuous
- joint right_leg_to_slave_right_axix4: type fixed -> continuous
- joint right_leg_to_slave_right_axix5: type fixed -> continuous
